File: Board/Rev1/pico-ice.kicad_pcb (KiCad board)
At the start: 4 copper layers, 22.9 x 61 mm, 99 parts, among them J1 USB_C_Receptacle_USB2.0, J2 Conn_02x20_Odd_Even, J3 Conn_02x20_Odd_Even, J4 PB_SEL, Q1 2N7002, SW1 PTS820 J25K SMTR LFS, SW2 PTS820 J25K SMTR LFS, U1 CL9293A12L5M, U2 W25Q32JVSSIQ, U3 RP2040, U4 CL9293A33L5M, U5 APS6404L-3SQN-SN, U6 ICE40UP5K-SG48ITR, U8 W25Q32JVSSIQ, Y1 12 MHz

Commit message: Minor changes to placement
Parts:
- J4: moved to B.Cu
- moved R14 26.7 mm to (66.2, 76.2), turned to 90 degrees
- moved D3 25.6 mm to (67.6, 76.2), turned to -90 degrees
- moved J4 8.95 mm to (72.4, 127.9)
Changed lines of the file:
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@@
   )
   (footprint "LED_SMD:LED_0603_1608Metric" (layer "F.Cu")
-    (at 75.4888 100.5332 90)
+    (at 67.564 76.2 -90)
     (descr "LED SMD 0603 (1608 Metric), square (rectangular) end terminal, IPC_7351 nominal, (Body size source: http://www.tortai-tech.com/upload/download/2011102023233369053.pdf), generated with kicad-footprint-generator")
     (tags "LED")
@@
     (fp_line (start -0.8 0.4) (end 0.8 0.4) (layer "F.Fab") (width 0.1))
     (fp_line (start -0.8 -0.1) (end -0.8 0.4) (layer "F.Fab") (width 0.1))
-    (pad "1" smd roundrect (at -0.7875 0 90) (size 0.875 0.95) (layers "F.Cu" "F.Paste" "F.Mask") (roundrect_rratio 0.25)
+    (pad "1" smd roundrect (at -0.7875 0 270) (size 0.875 0.95) (layers "F.Cu" "F.Paste" "F.Mask") (roundrect_rratio 0.25)
       (net 1 "GND") (pinfunction "K") (pintype "passive"))
-    (pad "2" smd roundrect (at 0.7875 0 90) (size 0.875 0.95) (layers "F.Cu" "F.Paste" "F.Mask") (roundrect_rratio 0.25)
+    (pad "2" smd roundrect (at 0.7875 0 270) (size 0.875 0.95) (layers "F.Cu" "F.Paste" "F.Mask") (roundrect_rratio 0.25)
       (net 27 "/ICE_DONE") (pinfunction "A") (pintype "passive"))
     (model "${KICAD6_3DMODEL_DIR}/LED_SMD.3dshapes/LED_0603_1608Metric.wrl"
@@
   )
   (footprint "Resistor_SMD:R_0402_1005Metric" (layer "F.Cu")
-    (at 77.1144 100.584)
+    (at 66.167 76.2 90)
     (descr "Resistor SMD 0402 (1005 Metric), square (rectangular) end terminal, IPC_7351 nominal, (Body size source: IPC-SM-782 page 72, https://www.pcb-3d.com/wordpress/wp-content/uploads/ipc-sm-782a_amendment_1_and_2.pdf), generated with kicad-footprint-generator")
     (tags "resistor")
@@
     (property "Supplier" "LCSC")
     (attr smd)
-    (fp_text reference "R14" (at 15.621 8.3312) (layer "F.SilkS") hide
+    (fp_text reference "R14" (at 15.621 8.3312 90) (layer "F.SilkS") hide
       (effects (font (size 0.889 0.889) (thickness 0.127)))
     )
-    (fp_text value "2.2K" (at 0 1.17) (layer "F.Fab")
+    (fp_text value "2.2K" (at 0 1.17 90) (layer "F.Fab")
       (effects (font (size 1 1) (thickness 0.15)))
     )
-    (fp_text user "${REFERENCE}" (at 0 0) (layer "F.Fab")
+    (fp_text user "${REFERENCE}" (at 0 0 90) (layer "F.Fab")
       (effects (font (size 0.26 0.26) (thickness 0.04)))
     )
@@
     (fp_line (start -0.525 0.27) (end -0.525 -0.27) (layer "F.Fab") (width 0.1))
     (fp_line (start 0.525 -0.27) (end 0.525 0.27) (layer "F.Fab") (width 0.1))
-    (pad "1" smd roundrect (at -0.51 0) (size 0.54 0.64) (layers "F.Cu" "F.Paste" "F.Mask") (roundrect_rratio 0.25)
+    (pad "1" smd roundrect (at -0.51 0 90) (size 0.54 0.64) (layers "F.Cu" "F.Paste" "F.Mask") (roundrect_rratio 0.25)
       (net 27 "/ICE_DONE") (pintype "passive"))
-    (pad "2" smd roundrect (at 0.51 0) (size 0.54 0.64) (layers "F.Cu" "F.Paste" "F.Mask") (roundrect_rratio 0.25)
+    (pad "2" smd roundrect (at 0.51 0 90) (size 0.54 0.64) (layers "F.Cu" "F.Paste" "F.Mask") (roundrect_rratio 0.25)
       (net 5 "+3V3") (pintype "passive"))
     (model "${KICAD6_3DMODEL_DIR}/Resistor_SMD.3dshapes/R_0402_1005Metric.wrl"
@@
     )
   )
-  (footprint "Jumper:SolderJumper-3_P1.3mm_Bridged12_RoundedPad1.0x1.5mm_NumberLabels" (layer "F.Cu")
-    (at 63.6016 129.5908)
-    (descr "SMD Solder 3-pad Jumper, 1x1.5mm rounded Pads, 0.3mm gap, pads 1-2 bridged with 1 copper strip, labeled with numbers")
-    (tags "net tie solder jumper bridged")
-    (property "Sheetfile" "pico-ice.kicad_sch")
-    (property "Sheetname" "")
-    (attr exclude_from_pos_files)
-    (fp_text reference "J4" (at 0 -1.8) (layer "F.SilkS")
-      (effects (font (size 1 1) (thickness 0.15)))
-    )
-    (fp_text value "PB_SEL" (at 0 1.9) (layer "F.Fab")
-      (effects (font (size 1 1) (thickness 0.15)))
-    )
-    (fp_text user "1" (at -2.6 0) (layer "F.SilkS")
-      (effects (font (size 1 1) (thickness 0.15)))
-    )
-    (fp_text user "3" (at 2.6 0) (layer "F.SilkS")
-      (effects (font (size 1 1) (thickness 0.15)))
-    )
-    (fp_poly (pts
-        (xy -0.9 -0.3)
-        (xy -0.4 -0.3)
-        (xy -0.4 0.3)
-        (xy -0.9 0.3)
-      ) (layer "F.Cu") (width 0) (fill solid))
-    (fp_line (start 1.4 1) (end -1.4 1) (layer "F.SilkS") (width 0.12))
-    (fp_line (start -1.4 -1) (end 1.4 -1) (layer "F.SilkS") (width 0.12))
-    (fp_line (start -2.05 0.3) (end -2.05 -0.3) (layer "F.SilkS") (width 0.12))
-    (fp_line (start 2.05 -0.3) (end 2.05 0.3) (layer "F.SilkS") (width 0.12))
-    (fp_arc (start 2.05 0.3) (mid 1.844975 0.794975) (end 1.35 1) (layer "F.SilkS") (width 0.12))
-    (fp_arc (start -2.05 -0.3) (mid -1.844975 -0.794975) (end -1.35 -1) (layer "F.SilkS") (width 0.12))
-    (fp_arc (start -1.35 1) (mid -1.844975 0.794975) (end -2.05 0.3) (layer "F.SilkS") (width 0.12))
-    (fp_arc (start 1.35 -1) (mid 1.844975 -0.794975) (end 2.05 -0.3) (layer "F.SilkS") (width 0.12))
-    (fp_line (start -2.3 -1.25) (end 2.3 -1.25) (layer "F.CrtYd") (width 0.05))
-    (fp_line (start 2.3 1.25) (end 2.3 -1.25) (layer "F.CrtYd") (width 0.05))
-    (fp_line (start 2.3 1.25) (end -2.3 1.25) (layer "F.CrtYd") (width 0.05))
-    (fp_line (start -2.3 -1.25) (end -2.3 1.25) (layer "F.CrtYd") (width 0.05))
-    (pad "1" smd custom (at -1.3 0) (size 1 0.5) (layers "F.Cu" "F.Mask")
-      (net 28 "/~{RESET}") (pinfunction "Pin_1") (pintype "passive") (zone_connect 2)
-      (options (clearance outline) (anchor rect))
-      (primitives
-        (gr_poly (pts
-            (xy 0.55 0.75)
-            (xy 0 0.75)
-            (xy 0 -0.75)
-            (xy 0.55 -0.75)
-          ) (width 0) (fill yes))
-            (gr_circle (center 0 0.25) (end 0.5 0.25) (width 0) (fill yes))
-            (gr_circle (center 0 -0.25) (end 0.5 -0.25) (width 0) (fill yes))
-      ))
-    (pad "2" smd rect (at 0 0) (size 1 1.5) (layers "F.Cu" "F.Mask")
-      (net 88 "Net-(J4-Pad2)") (pinfunction "Pin_2") (pintype "passive"))
-    (pad "3" smd custom (at 1.3 0) (size 1 0.5) (layers "F.Cu" "F.Mask")
-      (net 89 "/ADC2|PB") (pinfunction "Pin_3") (pintype "passive") (zone_connect 2)
-      (options (clearance outline) (anchor rect))
-      (primitives
-        (gr_circle (center 0 0.25) (end 0.5 0.25) (width 0) (fill yes))
-        (gr_circle (center 0 -0.25) (end 0.5 -0.25) (width 0) (fill yes))
-        (gr_poly (pts
-            (xy 0 0.75)
-            (xy -0.55 0.75)
-            (xy -0.55 -0.75)
-            (xy 0 -0.75)
-          ) (width 0) (fill yes))
-      ))
-  )
   (footprint "Capacitor_SMD:C_0402_1005Metric" (layer "F.Cu")
     (at 69.088 118.7958 -90)
@@
     )
   )
+  (footprint "Jumper:SolderJumper-3_P1.3mm_Bridged12_RoundedPad1.0x1.5mm_NumberLabels" (layer "B.Cu")
+    (at 72.39 127.889)
+    (descr "SMD Solder 3-pad Jumper, 1x1.5mm rounded Pads, 0.3mm gap, pads 1-2 bridged with 1 copper strip, labeled with numbers")
+    (tags "net tie solder jumper bridged")
+    (property "Sheetfile" "pico-ice.kicad_sch")
+    (property "Sheetname" "")
+    (attr exclude_from_pos_files)
+    (fp_text reference "J4" (at 0 1.8) (layer "B.SilkS")
+      (effects (font (size 1 1) (thickness 0.15)) (justify mirror))
+    )
+    (fp_text value "PB_SEL" (at 0 -1.9) (layer "B.Fab")
+      (effects (font (size 1 1) (thickness 0.15)) (justify mirror))
+    )
+    (fp_text user "1" (at -2.6 0) (layer "B.SilkS")
+      (effects (font (size 1 1) (thickness 0.15)) (justify mirror))
+    )
+    (fp_text user "3" (at 2.6 0) (layer "B.SilkS")
+      (effects (font (size 1 1) (thickness 0.15)) (justify mirror))
+    )
+    (fp_poly (pts
+        (xy -0.9 0.3)
+        (xy -0.4 0.3)
+        (xy -0.4 -0.3)
+        (xy -0.9 -0.3)
+      ) (layer "B.Cu") (width 0) (fill solid))
+    (fp_line (start 1.4 -1) (end -1.4 -1) (layer "B.SilkS") (width 0.12))
+    (fp_line (start -1.4 1) (end 1.4 1) (layer "B.SilkS") (width 0.12))
+    (fp_line (start -2.05 -0.3) (end -2.05 0.3) (layer "B.SilkS") (width 0.12))
+    (fp_line (start 2.05 0.3) (end 2.05 -0.3) (layer "B.SilkS") (width 0.12))
+    (fp_arc (start 1.35 -1) (mid 1.844975 -0.794975) (end 2.05 -0.3) (layer "B.SilkS") (width 0.12))
+    (fp_arc (start -1.35 1) (mid -1.844975 0.794975) (end -2.05 0.3) (layer "B.SilkS") (width 0.12))
+    (fp_arc (start -2.05 -0.3) (mid -1.844975 -0.794975) (end -1.35 -1) (layer "B.SilkS") (width 0.12))
+    (fp_arc (start 2.05 0.3) (mid 1.844975 0.794975) (end 1.35 1) (layer "B.SilkS") (width 0.12))
+    (fp_line (start -2.3 1.25) (end 2.3 1.25) (layer "B.CrtYd") (width 0.05))
+    (fp_line (start 2.3 -1.25) (end 2.3 1.25) (layer "B.CrtYd") (width 0.05))
+    (fp_line (start 2.3 -1.25) (end -2.3 -1.25) (layer "B.CrtYd") (width 0.05))
+    (fp_line (start -2.3 1.25) (end -2.3 -1.25) (layer "B.CrtYd") (width 0.05))
+    (pad "1" smd custom (at -1.3 0) (size 1 0.5) (layers "B.Cu" "B.Mask")
+      (net 28 "/~{RESET}") (pinfunction "Pin_1") (pintype "passive") (zone_connect 2)
+      (options (clearance outline) (anchor rect))
+      (primitives
+        (gr_poly (pts
+            (xy 0.55 -0.75)
+            (xy 0 -0.75)
+            (xy 0 0.75)
+            (xy 0.55 0.75)
+          ) (width 0) (fill yes))
+            (gr_circle (center 0 -0.25) (end 0.5 -0.25) (width 0) (fill yes))
+            (gr_circle (center 0 0.25) (end 0.5 0.25) (width 0) (fill yes))
+      ))
+    (pad "2" smd rect (at 0 0) (size 1 1.5) (layers "B.Cu" "B.Mask")
+      (net 88 "Net-(J4-Pad2)") (pinfunction "Pin_2") (pintype "passive"))
+    (pad "3" smd custom (at 1.3 0) (size 1 0.5) (layers "B.Cu" "B.Mask")
+      (net 89 "/ADC2|PB") (pinfunction "Pin_3") (pintype "passive") (zone_connect 2)
+      (options (clearance outline) (anchor rect))
+      (primitives
+        (gr_circle (center 0 -0.25) (end 0.5 -0.25) (width 0) (fill yes))
+        (gr_circle (center 0 0.25) (end 0.5 0.25) (width 0) (fill yes))
+        (gr_poly (pts
+            (xy 0 -0.75)
+            (xy -0.55 -0.75)
+            (xy -0.55 0.75)
+            (xy 0 0.75)
+          ) (width 0) (fill yes))
+      ))
+  )
   (footprint "Resistor_SMD:R_0402_1005Metric" (layer "B.Cu")
