File: Board/Rev1/pico-ice.kicad_pcb (KiCad board)
At the start: 4 copper layers, 22.9 x 61 mm, 99 parts, among them J1 USB_C_Receptacle_USB2.0, J2 Conn_02x20_Odd_Even, J3 Conn_02x20_Odd_Even, J4 PB_SEL, Q1 2N7002, SW1 PTS820 J25K SMTR LFS, SW2 PTS820 J25K SMTR LFS, U1 CL9293A12L5M, U2 W25Q32JVSSIQ, U3 RP2040, U4 CL9293A33L5M, U5 APS6404L-3SQN-SN, U6 ICE40UP5K-SG48ITR, U8 W25Q32JVSSIQ, Y1 12 MHz

Commit message: Finished the layout for a review.
Parts:
- moved LOGO1 46.6 mm to (75.1, 82.4), turned to 0 degrees
- moved LOGO2 24.4 mm to (72.6, 112.3)
- moved FID4 23.3 mm to (78.5, 132.8)
- moved FID3 21.1 mm to (78.5, 132.8)
- moved FID1 21.0 mm to (78.0, 81.3)
- moved RN1 15.9 mm to (69.8, 83.8), turned to 90 degrees
- moved LOGO3 15.8 mm to (69.7, 95.1)
- moved FID2 12.0 mm to (70.2, 77.2)
- moved FID6 11.8 mm to (66.3, 132.8)
- moved FID5 7.72 mm to (66.3, 132.8)
- moved C7 5.20 mm to (71.1, 102.0), turned to 0 degrees
- moved C37 4.51 mm to (69.4, 105.7), turned to 90 degrees
- moved C8 3.05 mm to (69.0, 119.3)
- moved R16 1.45 mm to (69.1, 107.7)
- moved R2 1.22 mm to (77.1, 120.2)
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Connections:
- J3 pad 24: unconnected-(J3-Pad24) -> /PICO_PMOD_B1
- J3 pad 26: unconnected-(J3-Pad26) -> /PICO_PMOD_B2
- J3 pad 28: unconnected-(J3-Pad28) -> /PICO_PMOD_B3
- J3 pad 30: unconnected-(J3-Pad30) -> /PICO_PMOD_B4
Routing:
- net +3V3: track 617.5 -> 60.3 mm, vias 42 -> 22
- net GND: track 470.7 -> 40.1 mm, vias 44 -> 31
- net /+3V3_STDBY: track 1.66 -> 77.9 mm, vias 4 -> 3
- net /SRAM_SS: track 0.25 -> 63.0 mm, vias 0 -> 3
- net /ICE_SSN: track 1.26 -> 63.4 mm, vias 0 -> 5
- net /ADC2|PB: track 0.00 -> 58.7 mm, vias 0 -> 2
- net /LED_B: track 24.0 -> 79.9 mm, vias 1 -> 5
- net /ICE_SCK: track 0.00 -> 55.2 mm, vias 0 -> 5
- net /~{ICE_RST}: track 0.00 -> 53.7 mm, vias 0 -> 4
- net /VIO_BANK_2: track 67.0 -> 14.9 mm, vias 4 -> 1
- net /LED_R: track 21.2 -> 73.3 mm, vias 0 -> 5
- net /ICE_27: track 1.02 -> 48.2 mm
- net /ICE_31: track 57.9 -> 10.8 mm, vias 3 -> 0
- net unconnected-(J3-Pad30): track 46.2 -> 0.00 mm, vias 2 -> 0
- net /ICE_SI: track 15.9 -> 60.1 mm, vias 1 -> 4
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- added copper zone on F.Cu, net VBUS
- added copper zone on F.Cu, net VDC
- added copper zone on In2.Cu, net VDC
- removed copper zone on B.Cu, net VBUS
