File: Board/Rev2/pico-ice.kicad_sch (KiCad schematic)
At the start: 99 parts, among them J1 USB_C_Receptacle_USB2.0, J2 Conn_02x20_Odd_Even, J3 Conn_02x20_Odd_Even, J4 PB_SEL, Q1 2N7002, SW1 PTS820 J25K SMTR LFS, SW2 PTS820 J25K SMTR LFS, U1 CL9293A12L5M, U2 W25Q32JVSSIQ, U3 RP2040, U4 CL9293A33L5M, U5 APS6404L-3SQN-SN, U6 ICE40UP5K-SG48ITR, U8 W25Q32JVSSIQ, Y1 12 MHz

Commit message: Added OSHW logo
Parts:
- added LOGO4: OSHW ID: US002140, OSHW_Certification:OSHW_Dual_0.1_Scale_2140, symbol MK11_PROG-rescue:TestPoint_Small-custom
Changed lines of the file:
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@@
     (stroke (width 0) (type default) (color 0 0 0 0))
   )
-  (polyline (pts (xy 300.355 259.715) (xy 300.355 260.35))
-    (stroke (width 0) (type default) (color 0 0 0 0))
-  )
   (wire (pts (xy 59.055 139.7) (xy 45.085 139.7))
     (stroke (width 0) (type default) (color 0 0 0 0))
@@
     (pin "2")
   )
+  (symbol (lib_id "MK11_PROG-rescue:TestPoint_Small-custom") (at 250.19 260.985 0) (unit 1)
+    (in_bom no) (on_board yes)
+    (property "Reference" "LOGO4" (id 0) (at 250.19 256.286 0))
+    (property "Value" "OSHW ID: US002140" (id 1) (at 250.19 258.5974 0))
+    (property "Footprint" "OSHW_Certification:OSHW_Dual_0.1_Scale_2140" (id 2) (at 255.27 260.985 0)
+      (effects (font (size 1.27 1.27)) hide)
+    )
+    (property "Datasheet" "~" (id 3) (at 255.27 260.985 0)
+      (effects (font (size 1.27 1.27)) hide)
+    )
+    (property "MPN" "DNP" (id 4) (at 250.19 260.985 0)
+      (effects (font (size 1.27 1.27)) hide)
+    )
+    (property "Digi-Key_PN" "DNP" (id 5) (at 250.19 260.985 0)
+      (effects (font (size 1.27 1.27)) hide)
+    )
+    (property "Manufacturer" "DNP" (id 6) (at 250.19 260.985 0)
+      (effects (font (size 1.27 1.27)) hide)
+    )
+  )
   (symbol (lib_id "UPduino_v3.0:power_+1V2") (at 132.715 55.88 0) (unit 1)
     (in_bom yes) (on_board yes)
@@
       (reference "LOGO3") (unit 1) (value "Pb free Logo") (footprint "CUSTOM:Pb free logo")
     )
+    (path "/de055fe0-26e3-4425-ac3c-584433236a2a"
+      (reference "LOGO4") (unit 1) (value "OSHW ID: US002140") (footprint "OSHW_Certification:OSHW_Dual_0.1_Scale_2140")
+    )
     (path "/049aa225-c9e7-467f-ab50-3f5e712805e5"
